File: project/wiscale.kicad_pcb (KiCad board)
At the start: 2 copper layers, 100 x 50 mm, 107 parts, among them J405 cell, J505 cell, J605 cell, J701 DS18B20, J801 DS18B20, J901 i2c, Q301 AO3401A, Q302 AO3401A, Q401 AO3401A, Q501 AO3401A, Q601 AO3401A, SW301 SW_SPDT, SW302 btn, U201 ESP-7(S) or ESP-12*, U301 BMS_USB_LiPo_Charger, U302 TPL5110, U401 HX711, U501 HX711, U601 HX711, U701 DS18B20Z, U702 DS18B20, U801 DS18B20Z, U802 DS18B20

Commit message: extracting load cell adapter to its own page
Parts:
- renumbered J405 to J401, J505 to J501, J605 to J601
Connections:
- SW301 pad : GND -> (no net)
- U701 pad 1: /MCU/1w -> unconnected-(U701-Pad1)
- U701 pad 8: GND -> unconnected-(U701-Pad8)
- U801 pad 1: /MCU/Charging -> unconnected-(U801-Pad1)
- U801 pad 8: GND -> unconnected-(U801-Pad8)
Changed lines of the file:
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@@
   (net 65 "Net-(R305-Pad2)")
   (net 66 "/PSU/_delay")
+  (net 67 "unconnected-(U701-Pad1)")
+  (net 68 "unconnected-(U701-Pad8)")
+  (net 69 "unconnected-(U801-Pad1)")
+  (net 70 "unconnected-(U801-Pad8)")
   (footprint "-local:JST_XH_S4B-XH-SM4-TB_1x04-1MP_P2.50mm_Horizontal" (layer "F.Cu")
     (at 139.2625 106.681843)
@@
     (property "Sheetname" "ADC3")
     (attr smd)
-    (fp_text reference "J605" (at 11.568393 1.970893 90 unlocked) (layer "F.SilkS")
+    (fp_text reference "J601" (at 11.568393 1.970893 90 unlocked) (layer "F.SilkS")
       (effects (font (size 0.8 0.8) (thickness 0.15)))
     )
@@
     (fp_line (start -3.35 1.6) (end 3.35 1.6) (layer "F.Fab") (width 0.1))
     (fp_line (start -1.2 3.15) (end -0.35 3.15) (layer "F.Fab") (width 0.1))
-    (pad "" smd rect (at 3.65 1.43 90) (size 1 0.8) (layers "F.Cu" "F.Paste" "F.Mask")
-      (net 3 "GND"))
+    (pad "" smd rect (at 3.65 1.43 90) (size 1 0.8) (layers "F.Cu" "F.Paste" "F.Mask"))
     (pad "" np_thru_hole circle (at 1.5 0.33 90) (size 0.9 0.9) (drill 0.9) (layers *.Cu *.Mask))
-    (pad "" smd rect (at -3.65 -0.78 90) (size 1 0.8) (layers "F.Cu" "F.Paste" "F.Mask")
-      (net 3 "GND"))
-    (pad "" smd rect (at -3.65 1.43 90) (size 1 0.8) (layers "F.Cu" "F.Paste" "F.Mask")
-      (net 3 "GND"))
-    (pad "" smd rect (at 3.65 -0.78 90) (size 1 0.8) (layers "F.Cu" "F.Paste" "F.Mask")
-      (net 3 "GND"))
+    (pad "" smd rect (at -3.65 -0.78 90) (size 1 0.8) (layers "F.Cu" "F.Paste" "F.Mask"))
+    (pad "" smd rect (at -3.65 1.43 90) (size 1 0.8) (layers "F.Cu" "F.Paste" "F.Mask"))
+    (pad "" smd rect (at 3.65 -0.78 90) (size 1 0.8) (layers "F.Cu" "F.Paste" "F.Mask"))
     (pad "" np_thru_hole circle (at -1.5 0.33 90) (size 0.9 0.9) (drill 0.9) (layers *.Cu *.Mask))
     (pad "1" smd rect (at -2.25 -1.43 90) (size 0.7 1.5) (layers "F.Cu" "F.Paste" "F.Mask")
@@
     (property "Sheetname" "PSU")
     (attr smd)
-    (fp_text reference "R308" (at -0.05 -1.375 unlocked) (layer "F.SilkS")
+    (fp_text reference "R308" (at -2.2825 -1.4625 unlocked) (layer "F.SilkS")
       (effects (font (size 0.8 0.8) (thickness 0.15)))
     )
@@
     (property "Sheetname" "ADC1")
     (attr smd)
-    (fp_text reference "J405" (at 11.568393 1.970893 90 unlocked) (layer "F.SilkS")
+    (fp_text reference "J401" (at 11.568393 1.970893 90 unlocked) (layer "F.SilkS")
       (effects (font (size 0.8 0.8) (thickness 0.15)))
     )
@@
     (fp_line (start -0.975 -2.45) (end 1.95 -2.45) (layer "F.Fab") (width 0.1))
     (pad "1" smd roundrect (at -2.475 -1.905 270) (size 1.95 0.6) (layers "F.Cu" "F.Paste" "F.Mask") (roundrect_rratio 0.25)
-      (net 30 "/MCU/Charging") (pinfunction "NC") (pintype "no_connect"))
+      (net 69 "unconnected-(U801-Pad1)") (pinfunction "NC") (pintype "no_connect"))
     (pad "2" smd roundrect (at -2.475 -0.635 270) (size 1.95 0.6) (layers "F.Cu" "F.Paste" "F.Mask") (roundrect_rratio 0.25)
       (net 55 "unconnected-(U801-Pad2)") (pinfunction "NC") (pintype "no_connect"))
@@
       (net 57 "unconnected-(U801-Pad7)") (pinfunction "NC") (pintype "no_connect"))
     (pad "8" smd roundrect (at 2.475 -1.905 270) (size 1.95 0.6) (layers "F.Cu" "F.Paste" "F.Mask") (roundrect_rratio 0.25)
-      (net 3 "GND") (pinfunction "NC") (pintype "no_connect"))
+      (net 70 "unconnected-(U801-Pad8)") (pinfunction "NC") (pintype "no_connect"))
     (model "${KICAD6_3DMODEL_DIR}/Package_SO.3dshapes/SOIC-8_3.9x4.9mm_P1.27mm.wrl"
       (offset (xyz 0 0 0))
@@
     (fp_line (start -0.975 -2.45) (end 1.95 -2.45) (layer "F.Fab") (width 0.1))
     (pad "1" smd roundrect (at -2.475 -1.905 270) (size 1.95 0.6) (layers "F.Cu" "F.Paste" "F.Mask") (roundrect_rratio 0.25)
-      (net 29 "/MCU/1w") (pinfunction "NC") (pintype "no_connect"))
+      (net 67 "unconnected-(U701-Pad1)") (pinfunction "NC") (pintype "no_connect"))
     (pad "2" smd roundrect (at -2.475 -0.635 270) (size 1.95 0.6) (layers "F.Cu" "F.Paste" "F.Mask") (roundrect_rratio 0.25)
       (net 52 "unconnected-(U701-Pad2)") (pinfunction "NC") (pintype "no_connect"))
@@
       (net 54 "unconnected-(U701-Pad7)") (pinfunction "NC") (pintype "no_connect"))
     (pad "8" smd roundrect (at 2.475 -1.905 270) (size 1.95 0.6) (layers "F.Cu" "F.Paste" "F.Mask") (roundrect_rratio 0.25)
-      (net 3 "GND") (pinfunction "NC") (pintype "no_connect"))
+      (net 68 "unconnected-(U701-Pad8)") (pinfunction "NC") (pintype "no_connect"))
     (model "${KICAD6_3DMODEL_DIR}/Package_SO.3dshapes/SOIC-8_3.9x4.9mm_P1.27mm.wrl"
       (offset (xyz 0 0 0))
@@
     (property "Sheetname" "ADC2")
     (attr smd)
-    (fp_text reference "J505" (at 11.568393 1.970893 90 unlocked) (layer "F.SilkS")
+    (fp_text reference "J501" (at 11.568393 1.970893 90 unlocked) (layer "F.SilkS")
       (effects (font (size 0.8 0.8) (thickness 0.15)))
     )
@@
     (property "Sheetname" "PSU")
     (attr smd)
-    (fp_text reference "U302" (at 0.725 2.125 unlocked) (layer "F.SilkS")
+    (fp_text reference "U302" (at 3.0325 2.125 unlocked) (layer "F.SilkS")
       (effects (font (size 0.8 0.8) (thickness 0.15)))
     )
@@
     (property "Sheetname" "PSU")
     (attr through_hole)
-    (fp_text reference "SW302" (at 1.3 -0.925 unlocked) (layer "F.SilkS")
+    (fp_text reference "SW302" (at 1.3 -3.4825 unlocked) (layer "F.SilkS")
       (effects (font (size 0.8 0.8) (thickness 0.15)))
     )

Commit message: various small improvements
Parts:
- SW301: footprint Button_Switch_SMD:SW_SPDT_PCM12 -> -local:SW_SPDT_PCM12
- moved LOGO102 7.42 mm to (135.0, 85.2)
- moved LOGO101 7.03 mm to (141.8, 85.7)
- moved R701 1.29 mm to (189.5, 107.5)
- moved R801 1.20 mm to (179.0, 107.5)
- moved kibuzzard-63766E45 0.58 mm to (105.5, 105.5)
- moved kibuzzard-63766E67 0.41 mm to (102.2, 72.8)
- moved kibuzzard-637D024E 0.25 mm to (124.9, 84.8)
Connections:
- net /MCU/ADC renamed /MCU/_adc
- net /MCU/RX renamed /MCU/_RX
- net Vusb renamed /PSU/_vusb
Routing:
- net /ADC1/Vcc: track 186.1 -> 190.6 mm
- net /MCU/1w: track 94.0 -> 96.7 mm
- net /MCU/Charging: track 97.8 -> 99.4 mm
Other:
- board text added: "1w1"
- board text added: "1w2"
- board text added: "ADC3"
- board text added: "D C Vc Gn"

Commit message: fixing bom, datasheets and adding link to repo
Parts:
- added G***: LOGO, -local:qr_wiscale_link_silkscreen, B.Cu at (186.0, 94.0)
- D201: value LED -> BLUE
- F301: value 1A -> PTC 1A
Other:
- board text added: "ID:"
- board text added: "SN:"

Commit message: adding usb port with ldo and diode options
Parts:
- added C307: 10u, Capacitor_SMD:C_0805_2012Metric_Pad1.18x1.45mm_HandSolder, F.Cu at (190.0, 95.4)
- added C308: 10u, Capacitor_SMD:C_0805_2012Metric_Pad1.18x1.45mm_HandSolder, F.Cu at (190.0, 88.8)
- added D301: 1N4148WL, Diode_SMD:D_SOD-123, F.Cu at (189.5, 97.8)
- added D302: 1N4148WL, Diode_SMD:D_SOD-123, F.Cu at (184.5, 97.8)
- added D303: GREEN, LED_SMD:LED_0805_2012Metric_Pad1.15x1.40mm_HandSolder, F.Cu at (196.4, 104.8)
- added J301: USB_POWER_IN, -local:USB_C_Receptacle_HRO_TYPE-C-31-M-12, F.Cu at (197.5, 93.2)
- added R309: 4k7, Resistor_SMD:R_0805_2012Metric_Pad1.20x1.40mm_HandSolder, F.Cu at (190.0, 91.0)
- added R310: 4k7, Resistor_SMD:R_0805_2012Metric_Pad1.20x1.40mm_HandSolder, F.Cu at (190.0, 93.2)
- added R311: 4k7, Resistor_SMD:R_0805_2012Metric_Pad1.20x1.40mm_HandSolder, F.Cu at (192.6, 104.8)
- added U303: AMS1117-3.3, Package_TO_SOT_SMD:SOT-223-3_TabPin2, F.Cu at (184.3, 92.2)
- moved G*** 56.0 mm to (132.5, 77.5)
- moved R302 1.40 mm to (196.4, 102.8)
- moved R301 1.39 mm to (192.6, 102.8)
Routing:
- net /PSU/_usb_vbus: track 0.00 -> 17.5 mm
- net Vbat: track 49.8 -> 63.9 mm
- net GND: track 62.9 -> 68.3 mm, vias 168 -> 181
- net /PSU/_cc1: track 0.00 -> 2.97 mm
- net /ADC1/Vcc: track 190.6 -> 193.4 mm
- net /PSU/_cc2: track 0.00 -> 2.64 mm
- net Net-(D303-Pad2): track 0.00 -> 1.78 mm
- net Net-(D301-Pad1): track 0.00 -> 1.74 mm
- net /PSU/_vusb: track 6.87 -> 6.26 mm
- net /MCU/Charging: track 99.4 -> 98.8 mm
- added copper zone on F.Cu, net Vbat

Commit message: removing metalization from the hole on the edge for manufacturing
Other:
- board text added: "JLCJLCJLCJLC"
Changed lines of the file:
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@@
     (property "Sheetname" "PSU")
     (property "exclude_from_bom" "")
-    (clearance 0.8)
     (attr smd exclude_from_bom)
     (fp_text reference "BT302" (at 16.55 -13.15 unlocked) (layer "F.SilkS")
@@
     (fp_rect (start 4 5) (end 42 -11) (layer "F.SilkS") (width 0.12) (fill none))
     (fp_rect (start -4.5 5.5) (end 42.5 -11.5) (layer "F.CrtYd") (width 0.05) (fill none))
-    (pad "" thru_hole oval (at 21.5 4.5 180) (size 5 2) (drill oval 4.5 1.6) (layers *.Mask "F.Cu" "In1.Cu" "B.Cu"))
+    (pad "" np_thru_hole oval (at 21.5 4.5 180) (size 4.5 1.6) (drill oval 4.5 1.6) (layers F&B.Cu *.Mask))
     (pad "" thru_hole oval (at 21.5 -10.5 180) (size 5 2) (drill oval 4.5 1.6) (layers *.Cu *.Mask))
     (pad "1" smd roundrect (at 0 0 180) (size 6.5 4) (layers "F.Cu" "F.Paste" "F.Mask") (roundrect_rratio 0.25)
@@
     (effects (font (size 0.8 0.8) (thickness 0.15)))
   )
+  (gr_text "JLCJLCJLCJLC" (at 155 67.5) (layer "F.SilkS")
+    (effects (font (size 1 1) (thickness 0.15)))
+  )
   (gr_text "ADC3" (at 148.9 85.7) (layer "F.SilkS")

Commit message: fixing mode select resistors values, related to #1
Parts:
- R203, R204, R205, R206: value 47k -> 10k

Commit message: consolidating RST with EN and adding a capacitor for stability. fixes #1
Parts:
- removed R204: 10k, Resistor_SMD:R_0805_2012Metric_Pad1.20x1.40mm_HandSolder
- removed kibuzzard-63766E45: G***, kibuzzard-63766E45
- added C204: 100n, Capacitor_SMD:C_0805_2012Metric_Pad1.18x1.45mm_HandSolder, F.Cu at (111.8, 112.2)
- added kibuzzard-63DFE172: G***, kibuzzard-63DFE172, F.Cu at (105.5, 105.5)
- moved R201 3.79 mm to (111.8, 108.4), turned to 90 degrees
Connections:
- U201 pad 3: /MCU/_EN -> /MCU/_RST
Routing:
- net /MCU/_RST: track 14.6 -> 25.2 mm
- net /MCU/_EN: track 8.94 -> 0.00 mm
- net /ADC1/Vcc: track 193.4 -> 192.3 mm
- net /MCU/_adc: track 17.6 -> 18.4 mm

Commit message: fixing charging detection divider, fixes #2
Parts:
- moved R301 3.80 mm to (196.4, 102.8), turned to 0 degrees
- moved R302 3.80 mm to (192.6, 102.8), turned to 0 degrees
Connections:
- R301 pad 1: /PSU/_vusb -> /MCU/Charging
- R301 pad 2: /MCU/Charging -> /PSU/_vusb
- R302 pad 2: /PSU/_vusb -> /MCU/Charging
Routing:
- net /MCU/Charging: track 98.2 -> 103.4 mm
- net /PSU/_vusb: track 6.26 -> 2.74 mm
Changed lines of the file:
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@@
   )
   (footprint "Resistor_SMD:R_0805_2012Metric_Pad1.20x1.40mm_HandSolder" (layer "F.Cu")
-    (at 192.6 102.8 180)
+    (at 196.4 102.8)
     (descr "Resistor SMD 0805 (2012 Metric), square (rectangular) end terminal, IPC_7351 nominal with elongated pad for handsoldering. (Body size source: IPC-SM-782 page 72, https://www.pcb-3d.com/wordpress/wp-content/uploads/ipc-sm-782a_amendment_1_and_2.pdf), generated with kicad-footprint-generator")
     (tags "resistor handsolder")
@@
     (property "Sheetname" "PSU")
     (attr smd)
-    (fp_text reference "R301" (at 3.4 0.4 unlocked) (layer "F.SilkS")
+    (fp_text reference "R301" (at 2.6 0.6 90 unlocked) (layer "F.SilkS")
       (effects (font (size 0.8 0.8) (thickness 0.15)))
     )
@@
     (fp_line (start 1 -0.625) (end 1 0.625) (layer "F.Fab") (width 0.1))
     (fp_line (start -1 -0.625) (end 1 -0.625) (layer "F.Fab") (width 0.1))
-    (pad "1" smd roundrect (at -1 0 180) (size 1.2 1.4) (layers "F.Cu" "F.Paste" "F.Mask") (roundrect_rratio 0.208333)
-      (net 58 "/PSU/_vusb") (pintype "passive"))
-    (pad "2" smd roundrect (at 1 0 180) (size 1.2 1.4) (layers "F.Cu" "F.Paste" "F.Mask") (roundrect_rratio 0.208333)
+    (pad "1" smd roundrect (at -1 0) (size 1.2 1.4) (layers "F.Cu" "F.Paste" "F.Mask") (roundrect_rratio 0.208333)
       (net 30 "/MCU/Charging") (pintype "passive"))
+    (pad "2" smd roundrect (at 1 0) (size 1.2 1.4) (layers "F.Cu" "F.Paste" "F.Mask") (roundrect_rratio 0.208333)
+      (net 58 "/PSU/_vusb") (pintype "passive"))
     (model "${KICAD6_3DMODEL_DIR}/Resistor_SMD.3dshapes/R_0805_2012Metric.wrl"
       (offset (xyz 0 0 0))
@@
   )
   (footprint "Resistor_SMD:R_0805_2012Metric_Pad1.20x1.40mm_HandSolder" (layer "F.Cu")
-    (at 196.4 102.8 180)
+    (at 192.6 102.8)
     (descr "Resistor SMD 0805 (2012 Metric), square (rectangular) end terminal, IPC_7351 nominal with elongated pad for handsoldering. (Body size source: IPC-SM-782 page 72, https://www.pcb-3d.com/wordpress/wp-content/uploads/ipc-sm-782a_amendment_1_and_2.pdf), generated with kicad-footprint-generator")
     (tags "resistor handsolder")
@@
     (property "Sheetname" "PSU")
     (attr smd)
-    (fp_text reference "R302" (at -2.6 -0.6 90 unlocked) (layer "F.SilkS")
+    (fp_text reference "R302" (at -3.2 -0.4 unlocked) (layer "F.SilkS")
       (effects (font (size 0.8 0.8) (thickness 0.15)))
     )
@@
     (fp_line (start 1 0.625) (end -1 0.625) (layer "F.Fab") (width 0.1))
     (fp_line (start -1 -0.625) (end 1 -0.625) (layer "F.Fab") (width 0.1))
-    (pad "1" smd roundrect (at -1 0 180) (size 1.2 1.4) (layers "F.Cu" "F.Paste" "F.Mask") (roundrect_rratio 0.208333)
+    (pad "1" smd roundrect (at -1 0) (size 1.2 1.4) (layers "F.Cu" "F.Paste" "F.Mask") (roundrect_rratio 0.208333)
       (net 3 "GND") (pintype "passive"))
-    (pad "2" smd roundrect (at 1 0 180) (size 1.2 1.4) (layers "F.Cu" "F.Paste" "F.Mask") (roundrect_rratio 0.208333)
-      (net 58 "/PSU/_vusb") (pintype "passive"))
+    (pad "2" smd roundrect (at 1 0) (size 1.2 1.4) (layers "F.Cu" "F.Paste" "F.Mask") (roundrect_rratio 0.208333)
+      (net 30 "/MCU/Charging") (pintype "passive"))
     (model "${KICAD6_3DMODEL_DIR}/Resistor_SMD.3dshapes/R_0805_2012Metric.wrl"
       (offset (xyz 0 0 0))
@@
   (via (at 162.8625 97.471607) (size 0.8) (drill 0.4) (layers "F.Cu" "B.Cu") (net 3))
   (via (at 125.92 110) (size 0.8) (drill 0.4) (layers "F.Cu" "B.Cu") (free) (net 3))
-  (via (at 197.4 102.8) (size 0.8) (drill 0.4) (layers "F.Cu" "B.Cu") (net 3))
   (via (at 145.42 114) (size 0.8) (drill 0.4) (layers "F.Cu" "B.Cu") (free) (net 3))
   (via (at 182.5 95.8) (size 0.8) (drill 0.4) (layers "F.Cu" "B.Cu") (net 3))
@@
   (via (at 109.92 93) (size 0.8) (drill 0.4) (layers "F.Cu" "B.Cu") (free) (net 3))
   (via (at 146.92 94.5) (size 0.8) (drill 0.4) (layers "F.Cu" "B.Cu") (free) (net 3))
+  (via (at 191.6 102.8) (size 0.8) (drill 0.4) (layers "F.Cu" "B.Cu") (net 3))
   (via (at 195.885 66.515) (size 0.8) (drill 0.4) (layers "F.Cu" "B.Cu") (net 3))
   (via (at 150.918393 100.927736) (size 0.8) (drill 0.4) (layers "F.Cu" "B.Cu") (net 3))
@@
   (segment (start 180.25 104.358214) (end 182.2675 102.340714) (width 0.5) (layer "F.Cu") (net 30))
   (segment (start 147.360892 111.5) (end 148.679049 110.181843) (width 0.5) (layer "F.Cu") (net 30))
+  (segment (start 189.659286 102.340714) (end 190.6 101.4) (width 0.5) (layer "F.Cu") (net 30))
   (segment (start 130.360893 111.5) (end 131.67905 110.181843) (width 0.5) (layer "F.Cu") (net 30))
   (segment (start 173.126612 106.976324) (end 173.126612 104.650714) (width 0.3) (layer "F.Cu") (net 30))
@@
   (segment (start 168.849822 110.785714) (end 170.766612 110.785714) (width 0.5) (layer "F.Cu") (net 30))
   (segment (start 113.42 102.25) (end 113.42 103.92) (width 0.5) (layer "F.Cu") (net 30))
-  (segment (start 182.2675 102.340714) (end 191.140714 102.340714) (width 0.5) (layer "F.Cu") (net 30))
+  (segment (start 193.2 101.4) (end 193.6 101.8) (width 0.5) (layer "F.Cu") (net 30))
   (segment (start 114.3 104.8) (end 116.33137 104.8) (width 0.5) (layer "F.Cu") (net 30))
   (segment (start 155.664108 111.5) (end 164.360892 111.5) (width 0.5) (layer "F.Cu") (net 30))
@@
   (segment (start 172.371612 109.185714) (end 172.371612 107.731324) (width 0.3) (layer "F.Cu") (net 30))
   (segment (start 172.371612 107.731324) (end 173.126612 106.976324) (width 0.3) (layer "F.Cu") (net 30))
+  (segment (start 195.4 102.8) (end 193.6 102.8) (width 0.5) (layer "F.Cu") (net 30))
   (segment (start 113.42 103.92) (end 114.3 104.8) (width 0.5) (layer "F.Cu") (net 30))
   (segment (start 138.664108 111.5) (end 147.360892 111.5) (width 0.5) (layer "F.Cu") (net 30))
-  (segment (start 191.140714 102.340714) (end 191.6 102.8) (width 0.5) (layer "F.Cu") (net 30))
+  (segment (start 193.6 101.8) (end 193.6 102.8) (width 0.5) (layer "F.Cu") (net 30))
   (segment (start 131.67905 110.181843) (end 137.345951 110.181843) (width 0.5) (layer "F.Cu") (net 30))
   (segment (start 172.411612 110.610714) (end 176.141612 110.610714) (width 0.3) (layer "F.Cu") (net 30))
   (segment (start 118.8225 107.922974) (end 118.8225 108.562737) (width 0.5) (layer "F.Cu") (net 30))
+  (segment (start 190.6 101.4) (end 193.2 101.4) (width 0.5) (layer "F.Cu") (net 30))
+  (segment (start 182.2675 102.340714) (end 189.659286 102.340714) (width 0.5) (layer "F.Cu") (net 30))
   (segment (start 176.141612 110.610714) (end 176.876612 109.875714) (width 0.3) (layer "F.Cu") (net 30))
   (segment (start 179 108.5) (end 177.624286 109.875714) (width 0.5) (layer "F.Cu") (net 30))
@@
   (segment (start 119.368393 85.185714) (end 128.936607 85.185714) (width 0.5) (layer "F.Cu") (net 47))
   (segment (start 130.1425 89.811607) (end 130.1425 90.531607) (width 0.5) (layer "F.Cu") (net 47))
-  (segment (start 196.35 100.25) (end 197.87 100.25) (width 0.5) (layer "F.Cu") (net 58))
-  (segment (start 193.6 102.8) (end 195.4 102.8) (width 0.5) (layer "F.Cu") (net 58))
-  (segment (start 195.4 102.8) (end 195.4 101.2) (width 0.5) (layer "F.Cu") (net 58))
-  (segment (start 195.4 101.2) (end 196.35 100.25) (width 0.5) (layer "F.Cu") (net 58))
+  (segment (start 197.87 100.25) (end 197.87 102.33) (width 1) (layer "F.Cu") (net 58))
+  (segment (start 197.87 102.33) (end 197.4 102.8) (width 1) (layer "F.Cu") (net 58))
   (segment (start 123.5525 88.485714) (end 121.7775 88.485714) (width 0.5) (layer "F.Cu") (net 59))
   (segment (start 158.016607 98.677736) (end 155.695179 98.677736) (width 0.5) (layer "F.Cu") (net 60))
