File: project/wiscale.kicad_pcb (KiCad board)
At the start: 2 copper layers, 100 x 50 mm, 118 parts, among them J301 USB_POWER_IN, J401 cell, J501 cell, J601 cell, J701 DS18B20, J801 DS18B20, J901 i2c, Q301 AO3401A, Q302 AO3401A, Q401 AO3401A, Q501 AO3401A, Q601 AO3401A, SW301 SW_SPDT, SW302 btn, U201 ESP-7(S) or ESP-12*, U301 BMS_USB_LiPo_Charger, U302 TPL5110, U303 AMS1117-3.3, U401 HX711, U501 HX711, U601 HX711, U701 DS18B20Z, U702 DS18B20, U801 DS18B20Z, U802 DS18B20

Commit message: connected LDO USB power with charger USB power, fixes #3
Connections:
- C307 pad 2: /PSU/_usb_vbus -> Vusb
- D301 pad 2: /PSU/_usb_vbus -> Vusb
- J301 pad A4: /PSU/_usb_vbus -> Vusb
- J301 pad A9: /PSU/_usb_vbus -> Vusb
- J301 pad B4: /PSU/_usb_vbus -> Vusb
- J301 pad B9: /PSU/_usb_vbus -> Vusb
- R301 pad 2: /PSU/_vusb -> Vusb
- U301 pad i1: /PSU/_vusb -> Vusb
- U303 pad 3: /PSU/_usb_vbus -> Vusb
Routing:
- net Vusb: track 0.00 -> 28.4 mm
- net /PSU/_usb_vbus: track 17.5 -> 0.00 mm
- net /PSU/_vusb: track 2.74 -> 0.00 mm
- net GND: vias 181 -> 191
