File: project/wiscale.kicad_pcb (KiCad board)
At the start: 2 copper layers, 100 x 50 mm, 118 parts, among them J301 USB_POWER_IN, J401 cell, J501 cell, J601 cell, J701 DS18B20, J801 DS18B20, J901 i2c, Q301 AO3401A, Q302 AO3401A, Q401 AO3401A, Q501 AO3401A, Q601 AO3401A, SW301 SW_SPDT, SW302 btn, U201 ESP-7(S) or ESP-12*, U301 BMS_USB_LiPo_Charger, U302 TPL5110, U303 AMS1117-3.3, U401 HX711, U501 HX711, U601 HX711, U701 DS18B20Z, U702 DS18B20, U801 DS18B20Z, U802 DS18B20

Commit message: adding more labels on silkscreen and bumping up version to 1.1
Parts:
- removed kibuzzard-63766E67: G***, kibuzzard-63766E67
- removed kibuzzard-63DFE172: G***, kibuzzard-63DFE172
- added kibuzzard-63DFF7BC: G***, kibuzzard-63DFF7BC, F.Cu at (102.2, 72.8)
- added kibuzzard-63DFF7CA: G***, kibuzzard-63DFF7CA, F.Cu at (105.5, 105.5)
Other:
- board text added: "-"
- board text added: "- +"
