File: project/wiscale.kicad_sch (KiCad schematic)
At the start: 6 parts

Commit message: extracting load cell adapter to its own page
Other:
- added sheet load cell adapter 4 to 1 (_load_cell_adapter.kicad_sch)
