File: project/_adc.kicad_sch (KiCad schematic)
At the start: 21 parts, among them J401 TL, J402 TR, J403 BL, J404 BR, J405 cell, Q401 AO3401A, U401 HX711

Commit message: extracting load cell adapter to its own page
Parts:
- removed J401: TL, Connector_JST:JST_XH_S3B-XH-A-1_1x03_P2.50mm_Horizontal, symbol Connector_Generic_MountingPin:Conn_01x03_MountingPin
- removed J402: TR, Connector_JST:JST_XH_S3B-XH-A-1_1x03_P2.50mm_Horizontal, symbol Connector_Generic_MountingPin:Conn_01x03_MountingPin
- removed J403: BL, Connector_JST:JST_XH_S3B-XH-A-1_1x03_P2.50mm_Horizontal, symbol Connector_Generic_MountingPin:Conn_01x03_MountingPin
- removed J404: BR, Connector_JST:JST_XH_S3B-XH-A-1_1x03_P2.50mm_Horizontal, symbol Connector_Generic_MountingPin:Conn_01x03_MountingPin
- renumbered J405 to J401

Commit message: fixing bom, datasheets and adding link to repo
Parts:
- J401: LCSC Part Number (none) -> C2905026; MPN (none) -> S4B-XH-SM4-TB(LF)(SN)
- Q401: LCSC Part Number (none) -> C347476; MPN (none) -> AO3401A
- U401: MPN (none) -> HX711
Changed lines of the file:
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@@
   (title_block
     (title "WiScale")
-    (date "2022-11-14")
+    (date "2022-11-24")
     (rev "1.0")
   )
@@
       (effects (font (size 1.27 1.27)) (justify left) hide)
     )
+    (property "LCSC Part Number" "C347476" (id 4) (at 171.45 77.47 0)
+      (effects (font (size 1.27 1.27)) hide)
+    )
+    (property "MPN" "AO3401A" (id 5) (at 171.45 77.47 0)
+      (effects (font (size 1.27 1.27)) hide)
+    )
     (pin "1")
     (pin "2")
@@
     )
     (property "LCSC Part Number" "C43656" (id 4) (at 198.12 133.35 0)
+      (effects (font (size 1.27 1.27)) hide)
+    )
+    (property "MPN" "HX711" (id 5) (at 179.07 101.6 0)
       (effects (font (size 1.27 1.27)) hide)
     )
@@
       (effects (font (size 1.27 1.27)) hide)
     )
-    (property "Datasheet" "~" (id 3) (at 101.6 102.87 0)
-      (effects (font (size 1.27 1.27)) hide)
-    )
+    (property "Datasheet" "https://datasheet.lcsc.com/lcsc/1810291321_JST-Sales-America-S4B-XH-SM4-TB-LF-SN_C161861.pdf" (id 3) (at 101.6 102.87 0)
+      (effects (font (size 1.27 1.27)) hide)
+    )
+    (property "LCSC Part Number" "C2905026" (id 4) (at 101.6 102.87 0)
+      (effects (font (size 1.27 1.27)) hide)
+    )
+    (property "MPN" "S4B-XH-SM4-TB(LF)(SN)" (id 5) (at 101.6 102.87 0)
+      (effects (font (size 1.27 1.27)) hide)
+    )
