File: project/_display.kicad_sch (KiCad schematic)
At the start: 4 parts, among them J901 i2c

Commit message: fixing bom, datasheets and adding link to repo
Other:
- title: (none) -> WiScale
Changed lines of the file:
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@@
 (kicad_sch (version 20211123) (generator eeschema)
   (paper "A4")
+  (title_block
+    (title "WiScale")
+    (date "2022-11-24")
+    (rev "1.0")
+  )
   (junction (at 153.67 96.52) (diameter 0) (color 0 0 0 0)
   )
