File: project/_load_cell_adapter.kicad_sch (KiCad schematic)
At the start: 5 parts, among them J1001 TL, J1002 TR, J1003 BL, J1004 BR, J1005 cell

Commit message: various small improvements
Other:
- moved on the sheet: J1001, J1002, J1004
Changed lines of the file:
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@@
 (kicad_sch (version 20211123) (generator eeschema)
   (paper "A4")
-  (wire (pts (xy 134.62 104.14) (xy 130.81 104.14))
+  (wire (pts (xy 130.81 134.62) (xy 143.51 134.62))
     (stroke (width 0) (type default) (color 0 0 0 0))
   )
-  (wire (pts (xy 153.67 60.96) (xy 130.81 60.96))
+  (wire (pts (xy 153.67 50.8) (xy 130.81 50.8))
     (stroke (width 0) (type default) (color 0 0 0 0))
   )
-  (wire (pts (xy 134.62 104.14) (xy 134.62 127))
+  (wire (pts (xy 135.89 48.26) (xy 135.89 76.2))
     (stroke (width 0) (type default) (color 0 0 0 0))
   )
-  (wire (pts (xy 153.67 106.68) (xy 130.81 106.68))
+  (wire (pts (xy 134.62 104.14) (xy 134.62 132.08))
     (stroke (width 0) (type default) (color 0 0 0 0))
   )
-  (wire (pts (xy 143.51 83.82) (xy 143.51 129.54))
+  (wire (pts (xy 130.81 78.74) (xy 143.51 78.74))
     (stroke (width 0) (type default) (color 0 0 0 0))
   )
-  (wire (pts (xy 135.89 58.42) (xy 130.81 58.42))
+  (wire (pts (xy 130.81 106.68) (xy 153.67 106.68))
     (stroke (width 0) (type default) (color 0 0 0 0))
   )
-  (wire (pts (xy 143.51 83.82) (xy 130.81 83.82))
+  (wire (pts (xy 143.51 78.74) (xy 143.51 134.62))
     (stroke (width 0) (type default) (color 0 0 0 0))
   )
-  (wire (pts (xy 134.62 127) (xy 130.81 127))
+  (wire (pts (xy 135.89 48.26) (xy 130.81 48.26))
     (stroke (width 0) (type default) (color 0 0 0 0))
   )
-  (wire (pts (xy 153.67 60.96) (xy 153.67 106.68))
+  (wire (pts (xy 134.62 132.08) (xy 130.81 132.08))
     (stroke (width 0) (type default) (color 0 0 0 0))
   )
-  (wire (pts (xy 143.51 129.54) (xy 130.81 129.54))
+  (wire (pts (xy 153.67 50.8) (xy 153.67 106.68))
     (stroke (width 0) (type default) (color 0 0 0 0))
   )
-  (wire (pts (xy 135.89 58.42) (xy 135.89 81.28))
+  (wire (pts (xy 130.81 76.2) (xy 135.89 76.2))
     (stroke (width 0) (type default) (color 0 0 0 0))
   )
-  (wire (pts (xy 135.89 81.28) (xy 130.81 81.28))
+  (wire (pts (xy 130.81 104.14) (xy 134.62 104.14))
     (stroke (width 0) (type default) (color 0 0 0 0))
   )
-  (label "_top_loop" (at 135.89 58.42 0)
+  (label "_top_loop" (at 135.89 48.26 0)
     (effects (font (size 1 1)) (justify left bottom))
   )
-  (label "_left_loop" (at 153.67 60.96 0)
+  (label "_left_loop" (at 153.67 50.8 0)
     (effects (font (size 1 1)) (justify left bottom))
   )
@@
     (effects (font (size 1.27 1.27)) (justify left bottom))
   )
-  (label "_right_loop" (at 143.51 83.82 0)
+  (label "_right_loop" (at 143.51 78.74 0)
     (effects (font (size 1 1)) (justify left bottom))
   )
@@
     (effects (font (size 1 1)) (justify left bottom))
   )
-  (label "E+" (at 130.81 124.46 0)
+  (label "E+" (at 130.81 129.54 0)
     (effects (font (size 1.27 1.27)) (justify left bottom))
   )
@@
     (effects (font (size 1.27 1.27)) (justify right bottom))
   )
-  (label "E-" (at 130.81 55.88 0)
+  (label "E-" (at 130.81 45.72 0)
     (effects (font (size 1.27 1.27)) (justify left bottom))
   )
@@
     (effects (font (size 1.27 1.27)) (justify right bottom))
   )
-  (label "S-" (at 130.81 78.74 0)
+  (label "S-" (at 130.81 73.66 0)
     (effects (font (size 1.27 1.27)) (justify left bottom))
   )
-  (symbol (lib_id "Connector_Generic_MountingPin:Conn_01x03_MountingPin") (at 125.73 127 0) (mirror y) (unit 1)
+  (symbol (lib_id "Connector_Generic_MountingPin:Conn_01x03_MountingPin") (at 125.73 132.08 0) (mirror y) (unit 1)
     (in_bom yes) (on_board no) (fields_autoplaced)
-    (property "Reference" "J1004" (id 0) (at 125.73 118.11 0))
-    (property "Value" "BR" (id 1) (at 125.73 120.65 0))
-    (property "Footprint" "Connector_JST:JST_XH_S3B-XH-A-1_1x03_P2.50mm_Horizontal" (id 2) (at 125.73 127 0)
+    (property "Reference" "J1004" (id 0) (at 125.73 123.19 0))
+    (property "Value" "BR" (id 1) (at 125.73 125.73 0))
+    (property "Footprint" "Connector_JST:JST_XH_S3B-XH-A-1_1x03_P2.50mm_Horizontal" (id 2) (at 125.73 132.08 0)
       (effects (font (size 1.27 1.27)) hide)
     )
-    (property "Datasheet" "~" (id 3) (at 125.73 127 0)
+    (property "Datasheet" "~" (id 3) (at 125.73 132.08 0)
       (effects (font (size 1.27 1.27)) hide)
     )
@@
     (pin "1")
   )
-  (symbol (lib_id "power:GND") (at 125.73 134.62 0) (unit 1)
+  (symbol (lib_id "power:GND") (at 125.73 139.7 0) (unit 1)
     (in_bom yes) (on_board yes)
-    (property "Reference" "#PWR01004" (id 0) (at 125.73 140.97 0)
+    (property "Reference" "#PWR01004" (id 0) (at 125.73 146.05 0)
       (effects (font (size 1.27 1.27)) hide)
     )
-    (property "Value" "GND" (id 1) (at 125.73 138.43 0))
-    (property "Footprint" "" (id 2) (at 125.73 134.62 0)
+    (property "Value" "GND" (id 1) (at 125.73 143.51 0))
+    (property "Footprint" "" (id 2) (at 125.73 139.7 0)
       (effects (font (size 1.27 1.27)) hide)
     )
-    (property "Datasheet" "" (id 3) (at 125.73 134.62 0)
+    (property "Datasheet" "" (id 3) (at 125.73 139.7 0)
       (effects (font (size 1.27 1.27)) hide)
     )
     (pin "1")
   )
-  (symbol (lib_id "Connector_Generic_MountingPin:Conn_01x03_MountingPin") (at 125.73 81.28 0) (mirror y) (unit 1)
+  (symbol (lib_id "Connector_Generic_MountingPin:Conn_01x03_MountingPin") (at 125.73 76.2 0) (mirror y) (unit 1)
     (in_bom yes) (on_board no)
-    (property "Reference" "J1002" (id 0) (at 125.73 72.39 0))
-    (property "Value" "TR" (id 1) (at 125.73 74.93 0))
-    (property "Footprint" "Connector_JST:JST_XH_S3B-XH-A-1_1x03_P2.50mm_Horizontal" (id 2) (at 125.73 81.28 0)
+    (property "Reference" "J1002" (id 0) (at 125.73 67.31 0))
+    (property "Value" "TR" (id 1) (at 125.73 69.85 0))
+    (property "Footprint" "Connector_JST:JST_XH_S3B-XH-A-1_1x03_P2.50mm_Horizontal" (id 2) (at 125.73 76.2 0)
       (effects (font (size 1.27 1.27)) hide)
     )
-    (property "Datasheet" "~" (id 3) (at 125.73 81.28 0)
+    (property "Datasheet" "~" (id 3) (at 125.73 76.2 0)
       (effects (font (size 1.27 1.27)) hide)
     )
@@
     (pin "MP")
   )
-  (symbol (lib_id "power:GND") (at 125.73 66.04 0) (unit 1)
+  (symbol (lib_id "power:GND") (at 125.73 55.88 0) (unit 1)
     (in_bom yes) (on_board yes)
-    (property "Reference" "#PWR01001" (id 0) (at 125.73 72.39 0)
+    (property "Reference" "#PWR01001" (id 0) (at 125.73 62.23 0)
       (effects (font (size 1.27 1.27)) hide)
     )
-    (property "Value" "GND" (id 1) (at 125.73 69.85 0))
-    (property "Footprint" "" (id 2) (at 125.73 66.04 0)
+    (property "Value" "GND" (id 1) (at 125.73 59.69 0))
+    (property "Footprint" "" (id 2) (at 125.73 55.88 0)
       (effects (font (size 1.27 1.27)) hide)
     )
-    (property "Datasheet" "" (id 3) (at 125.73 66.04 0)
+    (property "Datasheet" "" (id 3) (at 125.73 55.88 0)
       (effects (font (size 1.27 1.27)) hide)
     )
@@
     (pin "MP")
   )
-  (symbol (lib_id "power:GND") (at 125.73 88.9 0) (unit 1)
+  (symbol (lib_id "power:GND") (at 125.73 83.82 0) (unit 1)
     (in_bom yes) (on_board yes)
-    (property "Reference" "#PWR01002" (id 0) (at 125.73 95.25 0)
+    (property "Reference" "#PWR01002" (id 0) (at 125.73 90.17 0)
       (effects (font (size 1.27 1.27)) hide)
     )
-    (property "Value" "GND" (id 1) (at 125.73 92.71 0))
-    (property "Footprint" "" (id 2) (at 125.73 88.9 0)
+    (property "Value" "GND" (id 1) (at 125.73 87.63 0))
+    (property "Footprint" "" (id 2) (at 125.73 83.82 0)
       (effects (font (size 1.27 1.27)) hide)
     )
-    (property "Datasheet" "" (id 3) (at 125.73 88.9 0)
+    (property "Datasheet" "" (id 3) (at 125.73 83.82 0)
       (effects (font (size 1.27 1.27)) hide)
     )
     (pin "1")
   )
-  (symbol (lib_id "Connector_Generic_MountingPin:Conn_01x03_MountingPin") (at 125.73 58.42 0) (mirror y) (unit 1)
+  (symbol (lib_id "Connector_Generic_MountingPin:Conn_01x03_MountingPin") (at 125.73 48.26 0) (mirror y) (unit 1)
     (in_bom yes) (on_board no) (fields_autoplaced)
-    (property "Reference" "J1001" (id 0) (at 125.73 49.53 0))
-    (property "Value" "TL" (id 1) (at 125.73 52.07 0))
-    (property "Footprint" "Connector_JST:JST_XH_S3B-XH-A-1_1x03_P2.50mm_Horizontal" (id 2) (at 125.73 58.42 0)
+    (property "Reference" "J1001" (id 0) (at 125.73 39.37 0))
+    (property "Value" "TL" (id 1) (at 125.73 41.91 0))
+    (property "Footprint" "Connector_JST:JST_XH_S3B-XH-A-1_1x03_P2.50mm_Horizontal" (id 2) (at 125.73 48.26 0)
       (effects (font (size 1.27 1.27)) hide)
     )
-    (property "Datasheet" "~" (id 3) (at 125.73 58.42 0)
+    (property "Datasheet" "~" (id 3) (at 125.73 48.26 0)
       (effects (font (size 1.27 1.27)) hide)
     )

Commit message: fixing bom, datasheets and adding link to repo
Parts:
- J1005: LCSC Part Number (none) -> C2905026; MPN (none) -> S4B-XH-SM4-TB(LF)(SN)
Other:
- title: (none) -> WiScale
Changed lines of the file:
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@@
 (kicad_sch (version 20211123) (generator eeschema)
   (paper "A4")
+  (title_block
+    (title "WiScale")
+    (date "2022-11-24")
+    (rev "1.0")
+  )
   (wire (pts (xy 130.81 134.62) (xy 143.51 134.62))
     (stroke (width 0) (type default) (color 0 0 0 0))
@@
       (effects (font (size 1.27 1.27)) hide)
     )
-    (property "Datasheet" "~" (id 3) (at 175.26 87.63 0)
-      (effects (font (size 1.27 1.27)) hide)
-    )
+    (property "Datasheet" "https://datasheet.lcsc.com/lcsc/1810291321_JST-Sales-America-S4B-XH-SM4-TB-LF-SN_C161861.pdf" (id 3) (at 175.26 87.63 0)
+      (effects (font (size 1.27 1.27)) hide)
+    )
+    (property "LCSC Part Number" "C2905026" (id 4) (at 175.26 87.63 0)
+      (effects (font (size 1.27 1.27)) hide)
+    )
+    (property "MPN" "S4B-XH-SM4-TB(LF)(SN)" (id 5) (at 175.26 87.63 0)
+      (effects (font (size 1.27 1.27)) hide)
+    )
