File: project/_mcu.kicad_sch (KiCad schematic)
At the start: 12 parts, among them U201 ESP-7(S) or ESP-12*

Commit message: extracting load cell adapter to its own page
Parts:
- D201: footprint (none) -> LED_SMD:LED_0805_2012Metric_Pad1.15x1.40mm_HandSolder
Changed lines of the file:
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@@
       (effects (font (size 1.27 1.27)) (justify right))
     )
-    (property "Footprint" "" (id 2) (at 203.2 92.71 0)
+    (property "Footprint" "LED_SMD:LED_0805_2012Metric_Pad1.15x1.40mm_HandSolder" (id 2) (at 203.2 92.71 0)
       (effects (font (size 1.27 1.27)) hide)
     )

Commit message: various small improvements
Connections:
- net ADC renamed _adc
- net RX renamed _RX
Other:
- moved on the sheet: C201, D201, R201, R202, R207
Changed lines of the file:
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@@
   (junction (at 156.21 78.74) (diameter 0) (color 0 0 0 0)
   )
-  (junction (at 76.2 99.06) (diameter 0) (color 0 0 0 0)
+  (junction (at 83.82 96.52) (diameter 0) (color 0 0 0 0)
   )
   (junction (at 130.81 58.42) (diameter 0) (color 0 0 0 0)
   )
-  (junction (at 76.2 91.44) (diameter 0) (color 0 0 0 0)
+  (junction (at 83.82 88.9) (diameter 0) (color 0 0 0 0)
   )
   (junction (at 100.33 78.74) (diameter 0) (color 0 0 0 0)
   )
+  (junction (at 88.9 88.9) (diameter 0) (color 0 0 0 0)
+  )
   (junction (at 130.81 66.04) (diameter 0) (color 0 0 0 0)
   )
   (no_connect (at 142.24 81.28))
+  (wire (pts (xy 142.24 86.36) (xy 185.42 86.36))
+    (stroke (width 0) (type default) (color 0 0 0 0))
+  )
   (wire (pts (xy 158.75 83.82) (xy 142.24 83.82))
     (stroke (width 0) (type default) (color 0 0 0 0))
@@
     (stroke (width 0) (type default) (color 0 0 0 0))
   )
-  (wire (pts (xy 203.2 78.74) (xy 203.2 81.28))
+  (wire (pts (xy 185.42 63.5) (xy 185.42 66.04))
     (stroke (width 0) (type default) (color 0 0 0 0))
   )
@@
     (stroke (width 0) (type default) (color 0 0 0 0))
   )
-  (wire (pts (xy 76.2 91.44) (xy 81.28 91.44))
+  (wire (pts (xy 83.82 88.9) (xy 88.9 88.9))
     (stroke (width 0) (type default) (color 0 0 0 0))
   )
@@
     (stroke (width 0) (type default) (color 0 0 0 0))
   )
-  (wire (pts (xy 203.2 101.6) (xy 203.2 96.52))
+  (wire (pts (xy 185.42 86.36) (xy 185.42 81.28))
     (stroke (width 0) (type default) (color 0 0 0 0))
   )
@@
     (stroke (width 0) (type default) (color 0 0 0 0))
   )
-  (wire (pts (xy 76.2 99.06) (xy 81.28 99.06))
+  (wire (pts (xy 83.82 96.52) (xy 88.9 96.52))
     (stroke (width 0) (type default) (color 0 0 0 0))
   )
@@
     (stroke (width 0) (type default) (color 0 0 0 0))
   )
+  (wire (pts (xy 88.9 88.9) (xy 111.76 88.9))
+    (stroke (width 0) (type default) (color 0 0 0 0))
+  )
   (wire (pts (xy 100.33 73.66) (xy 100.33 78.74))
     (stroke (width 0) (type default) (color 0 0 0 0))
@@
     (stroke (width 0) (type default) (color 0 0 0 0))
   )
-  (label "ADC" (at 111.76 88.9 180)
-    (effects (font (size 1.27 1.27)) (justify right bottom))
-  )
-  (label "ADC" (at 78.74 91.44 0)
-    (effects (font (size 1.27 1.27)) (justify left bottom))
+  (label "_adc" (at 109.22 88.9 0)
+    (effects (font (size 0.5 0.5)) (justify left bottom))
   )
   (label "_RST" (at 109.22 78.74 0)
@@
     (effects (font (size 0.5 0.5)) (justify left bottom))
   )
-  (label "RX" (at 142.24 86.36 0)
-    (effects (font (size 1.27 1.27)) (justify left bottom))
-  )
-  (label "RX" (at 203.2 101.6 0)
-    (effects (font (size 1.27 1.27)) (justify left bottom))
-  )
-  (hierarchical_label "Vcc" (shape input) (at 76.2 83.82 90)
+  (label "_RX" (at 142.24 86.36 0)
+    (effects (font (size 0.5 0.5)) (justify left bottom))
+  )
+  (hierarchical_label "Vcc" (shape input) (at 83.82 81.28 90)
     (effects (font (size 1.27 1.27)) (justify left))
   )
@@
     (effects (font (size 1.27 1.27)) (justify left))
   )
-  (hierarchical_label "Vcc" (shape input) (at 203.2 78.74 90)
+  (hierarchical_label "Vcc" (shape input) (at 185.42 63.5 90)
     (effects (font (size 1.27 1.27)) (justify left))
   )
@@
     (pin "2")
   )
-  (symbol (lib_id "Device:R") (at 76.2 87.63 180) (unit 1)
-    (in_bom yes) (on_board yes)
-    (property "Reference" "R201" (id 0) (at 73.66 87.63 90))
-    (property "Value" "180k" (id 1) (at 76.2 87.63 90))
-    (property "Footprint" "Resistor_SMD:R_0805_2012Metric_Pad1.20x1.40mm_HandSolder" (id 2) (at 77.978 87.63 90)
-      (effects (font (size 1.27 1.27)) hide)
-    )
-    (property "Datasheet" "~" (id 3) (at 76.2 87.63 0)
+  (symbol (lib_id "Device:R") (at 83.82 85.09 180) (unit 1)
+    (in_bom yes) (on_board yes)
+    (property "Reference" "R201" (id 0) (at 81.28 85.09 90))
+    (property "Value" "180k" (id 1) (at 83.82 85.09 90))
+    (property "Footprint" "Resistor_SMD:R_0805_2012Metric_Pad1.20x1.40mm_HandSolder" (id 2) (at 85.598 85.09 90)
+      (effects (font (size 1.27 1.27)) hide)
+    )
+    (property "Datasheet" "~" (id 3) (at 83.82 85.09 0)
       (effects (font (size 1.27 1.27)) hide)
     )
@@
     (pin "1")
   )
-  (symbol (lib_id "Device:R") (at 76.2 95.25 180) (unit 1)
-    (in_bom yes) (on_board yes)
-    (property "Reference" "R202" (id 0) (at 73.66 95.25 90))
-    (property "Value" "47k" (id 1) (at 76.2 95.25 90))
-    (property "Footprint" "Resistor_SMD:R_0805_2012Metric_Pad1.20x1.40mm_HandSolder" (id 2) (at 77.978 95.25 90)
-      (effects (font (size 1.27 1.27)) hide)
-    )
-    (property "Datasheet" "~" (id 3) (at 76.2 95.25 0)
+  (symbol (lib_id "Device:R") (at 83.82 92.71 180) (unit 1)
+    (in_bom yes) (on_board yes)
+    (property "Reference" "R202" (id 0) (at 81.28 92.71 90))
+    (property "Value" "47k" (id 1) (at 83.82 92.71 90))
+    (property "Footprint" "Resistor_SMD:R_0805_2012Metric_Pad1.20x1.40mm_HandSolder" (id 2) (at 85.598 92.71 90)
+      (effects (font (size 1.27 1.27)) hide)
+    )
+    (property "Datasheet" "~" (id 3) (at 83.82 92.71 0)
       (effects (font (size 1.27 1.27)) hide)
     )
@@
     (pin "2")
   )
-  (symbol (lib_id "Device:LED") (at 203.2 92.71 90) (unit 1)
+  (symbol (lib_id "Device:LED") (at 185.42 77.47 90) (unit 1)
     (in_bom yes) (on_board yes) (fields_autoplaced)
-    (property "Reference" "D201" (id 0) (at 207.01 93.0274 90)
-      (effects (font (size 1.27 1.27)) (justify right))
-    )
-    (property "Value" "LED" (id 1) (at 207.01 95.5674 90)
-      (effects (font (size 1.27 1.27)) (justify right))
-    )
-    (property "Footprint" "LED_SMD:LED_0805_2012Metric_Pad1.15x1.40mm_HandSolder" (id 2) (at 203.2 92.71 0)
-      (effects (font (size 1.27 1.27)) hide)
-    )
-    (property "Datasheet" "~" (id 3) (at 203.2 92.71 0)
+    (property "Reference" "D201" (id 0) (at 189.23 77.7874 90)
+      (effects (font (size 1.27 1.27)) (justify right))
+    )
+    (property "Value" "LED" (id 1) (at 189.23 80.3274 90)
+      (effects (font (size 1.27 1.27)) (justify right))
+    )
+    (property "Footprint" "LED_SMD:LED_0805_2012Metric_Pad1.15x1.40mm_HandSolder" (id 2) (at 185.42 77.47 0)
+      (effects (font (size 1.27 1.27)) hide)
+    )
+    (property "Datasheet" "~" (id 3) (at 185.42 77.47 0)
       (effects (font (size 1.27 1.27)) hide)
     )
@@
     (pin "2")
   )
-  (symbol (lib_id "power:GND") (at 76.2 99.06 0) (unit 1)
-    (in_bom yes) (on_board yes)
-    (property "Reference" "#PWR0201" (id 0) (at 76.2 105.41 0)
-      (effects (font (size 1.27 1.27)) hide)
-    )
-    (property "Value" "GND" (id 1) (at 76.2 102.87 0))
-    (property "Footprint" "" (id 2) (at 76.2 99.06 0)
-      (effects (font (size 1.27 1.27)) hide)
-    )
-    (property "Datasheet" "" (id 3) (at 76.2 99.06 0)
+  (symbol (lib_id "power:GND") (at 83.82 96.52 0) (unit 1)
+    (in_bom yes) (on_board yes)
+    (property "Reference" "#PWR0201" (id 0) (at 83.82 102.87 0)
+      (effects (font (size 1.27 1.27)) hide)
+    )
+    (property "Value" "GND" (id 1) (at 83.82 100.33 0))
+    (property "Footprint" "" (id 2) (at 83.82 96.52 0)
+      (effects (font (size 1.27 1.27)) hide)
+    )
+    (property "Datasheet" "" (id 3) (at 83.82 96.52 0)
       (effects (font (size 1.27 1.27)) hide)
     )
@@
     (pin "2")
   )
-  (symbol (lib_id "Device:C") (at 81.28 95.25 180) (unit 1)
-    (in_bom yes) (on_board yes) (fields_autoplaced)
-    (property "Reference" "C201" (id 0) (at 85.09 93.9799 0)
-      (effects (font (size 1.27 1.27)) (justify right))
-    )
-    (property "Value" "100n" (id 1) (at 85.09 96.5199 0)
-      (effects (font (size 1.27 1.27)) (justify right))
-    )
-    (property "Footprint" "Capacitor_SMD:C_0805_2012Metric_Pad1.18x1.45mm_HandSolder" (id 2) (at 80.3148 91.44 0)
-      (effects (font (size 1.27 1.27)) hide)
-    )
-    (property "Datasheet" "~" (id 3) (at 81.28 95.25 0)
-      (effects (font (size 1.27 1.27)) hide)
-    )
-    (pin "1")
-    (pin "2")
-  )
-  (symbol (lib_id "Device:R") (at 203.2 85.09 180) (unit 1)
-    (in_bom yes) (on_board yes)
-    (property "Reference" "R207" (id 0) (at 200.66 85.09 90))
-    (property "Value" "100" (id 1) (at 203.2 85.09 90))
-    (property "Footprint" "Resistor_SMD:R_0805_2012Metric_Pad1.20x1.40mm_HandSolder" (id 2) (at 204.978 85.09 90)
-      (effects (font (size 1.27 1.27)) hide)
-    )
-    (property "Datasheet" "~" (id 3) (at 203.2 85.09 0)
-      (effects (font (size 1.27 1.27)) hide)
-    )
+  (symbol (lib_id "Device:C") (at 88.9 92.71 180) (unit 1)
+    (in_bom yes) (on_board yes)
+    (property "Reference" "C201" (id 0) (at 90.17 90.17 0)
+      (effects (font (size 1.27 1.27)) (justify right))
+    )
+    (property "Value" "100n" (id 1) (at 90.17 95.25 0)
+      (effects (font (size 1.27 1.27)) (justify right))
+    )
+    (property "Footprint" "Capacitor_SMD:C_0805_2012Metric_Pad1.18x1.45mm_HandSolder" (id 2) (at 87.9348 88.9 0)
+      (effects (font (size 1.27 1.27)) hide)
+    )
+    (property "Datasheet" "~" (id 3) (at 88.9 92.71 0)
+      (effects (font (size 1.27 1.27)) hide)
+    )
+    (pin "1")
+    (pin "2")
+  )
+  (symbol (lib_id "Device:R") (at 185.42 69.85 180) (unit 1)
+    (in_bom yes) (on_board yes)
+    (property "Reference" "R207" (id 0) (at 182.88 69.85 90))
+    (property "Value" "100" (id 1) (at 185.42 69.85 90))
+    (property "Footprint" "Resistor_SMD:R_0805_2012Metric_Pad1.20x1.40mm_HandSolder" (id 2) (at 187.198 69.85 90)
+      (effects (font (size 1.27 1.27)) hide)
+    )
+    (property "Datasheet" "~" (id 3) (at 185.42 69.85 0)
+      (effects (font (size 1.27 1.27)) hide)
+    )

Commit message: fixing bom, datasheets and adding link to repo
Parts:
- D201: value LED -> BLUE; LCSC Part Number (none) -> C965817; MPN (none) -> XL-2012UBC
- U201: LCSC Part Number (none) -> C89297; MPN (none) -> ESP-12E
Changed lines of the file:
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@@
   (title_block
     (title "WiScale")
-    (date "2022-11-14")
+    (date "2022-11-24")
     (rev "1.0")
   )
@@
       (effects (font (size 1.27 1.27)) (justify right))
     )
-    (property "Value" "LED" (id 1) (at 189.23 80.3274 90)
+    (property "Value" "BLUE" (id 1) (at 189.23 80.3274 90)
       (effects (font (size 1.27 1.27)) (justify right))
     )
@@
       (effects (font (size 1.27 1.27)) hide)
     )
-    (property "Datasheet" "~" (id 3) (at 185.42 77.47 0)
+    (property "Datasheet" "https://datasheet.lcsc.com/lcsc/2211030000_XINGLIGHT-XL-2012UBC_C965817.pdf" (id 3) (at 185.42 77.47 0)
+      (effects (font (size 1.27 1.27)) hide)
+    )
+    (property "LCSC Part Number" "C965817" (id 4) (at 185.42 77.47 0)
+      (effects (font (size 1.27 1.27)) hide)
+    )
+    (property "MPN" "XL-2012UBC" (id 5) (at 185.42 77.47 0)
       (effects (font (size 1.27 1.27)) hide)
     )
@@
       (effects (font (size 1.27 1.27)) hide)
     )
-    (property "Datasheet" "" (id 3) (at 118.11 91.44 0)
-      (effects (font (size 1.27 1.27)) hide)
-    )
+    (property "Datasheet" "https://www.espressif.com/sites/default/files/documentation/0a-esp8266ex_datasheet_en.pdf" (id 3) (at 118.11 91.44 0)
+      (effects (font (size 1.27 1.27)) hide)
+    )
+    (property "LCSC Part Number" "C89297" (id 4) (at 127 93.98 0)
+      (effects (font (size 1.27 1.27)) hide)
+    )
+    (property "MPN" "ESP-12E" (id 5) (at 127 93.98 0)
+      (effects (font (size 1.27 1.27)) hide)
+    )

Commit message: fixing mode select resistors values, related to #1
Parts:
- R203, R204, R205, R206: value 47k -> 10k
Changed lines of the file:
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@@
+    (stroke (width 0) (type default) (color 0 0 0 0))
+  )
+  (wire (pts (xy 158.75 91.44) (xy 142.24 91.44))
+    (stroke (width 0) (type default) (color 0 0 0 0))
+  )
+  (wire (pts (xy 142.24 88.9) (xy 158.75 88.9))
+    (stroke (width 0) (type default) (color 0 0 0 0))
+  )
+  (wire (pts (xy 158.75 78.74) (xy 156.21 78.74))
+    (stroke (width 0) (type default) (color 0 0 0 0))
+  )
+  (wire (pts (xy 142.24 99.06) (xy 158.75 99.06))
+    (stroke (width 0) (type default) (color 0 0 0 0))
+  )
+  (wire (pts (xy 158.75 93.98) (xy 142.24 93.98))
+    (stroke (width 0) (type default) (color 0 0 0 0))
+  )
+  (wire (pts (xy 83.82 88.9) (xy 88.9 88.9))
+    (stroke (width 0) (type default) (color 0 0 0 0))
+  )
+  (wire (pts (xy 158.75 101.6) (xy 156.21 101.6))
+    (stroke (width 0) (type default) (color 0 0 0 0))
+  )
+  (wire (pts (xy 140.97 58.42) (xy 130.81 58.42))
+    (stroke (width 0) (type default) (color 0 0 0 0))
+  )
+  (wire (pts (xy 130.81 58.42) (xy 127 58.42))
+    (stroke (width 0) (type default) (color 0 0 0 0))
+  )
+  (wire (pts (xy 107.95 83.82) (xy 111.76 83.82))
+    (stroke (width 0) (type default) (color 0 0 0 0))
+  )
+  (wire (pts (xy 185.42 86.36) (xy 185.42 81.28))
+    (stroke (width 0) (type default) (color 0 0 0 0))
+  )
+  (wire (pts (xy 156.21 78.74) (xy 142.24 78.74))
+    (stroke (width 0) (type default) (color 0 0 0 0))
+  )
+  (wire (pts (xy 100.33 63.5) (xy 100.33 78.74))
     (stroke (width 0) (type default) (color 0 0 0 0))
   )
@@
     (stroke (width 0) (type default) (color 0 0 0 0))
   )
-  (wire (pts (xy 158.75 91.44) (xy 142.24 91.44))
-    (stroke (width 0) (type default) (color 0 0 0 0))
-  )
-  (wire (pts (xy 142.24 88.9) (xy 158.75 88.9))
-    (stroke (width 0) (type default) (color 0 0 0 0))
-  )
-  (wire (pts (xy 158.75 78.74) (xy 156.21 78.74))
-    (stroke (width 0) (type default) (color 0 0 0 0))
-  )
-  (wire (pts (xy 142.24 99.06) (xy 158.75 99.06))
-    (stroke (width 0) (type default) (color 0 0 0 0))
-  )
-  (wire (pts (xy 158.75 93.98) (xy 142.24 93.98))
-    (stroke (width 0) (type default) (color 0 0 0 0))
-  )
-  (wire (pts (xy 83.82 88.9) (xy 88.9 88.9))
-    (stroke (width 0) (type default) (color 0 0 0 0))
-  )
-  (wire (pts (xy 158.75 101.6) (xy 156.21 101.6))
-    (stroke (width 0) (type default) (color 0 0 0 0))
-  )
-  (wire (pts (xy 140.97 58.42) (xy 130.81 58.42))
-    (stroke (width 0) (type default) (color 0 0 0 0))
-  )
-  (wire (pts (xy 130.81 58.42) (xy 127 58.42))
-    (stroke (width 0) (type default) (color 0 0 0 0))
-  )
-  (wire (pts (xy 107.95 83.82) (xy 111.76 83.82))
-    (stroke (width 0) (type default) (color 0 0 0 0))
-  )
-  (wire (pts (xy 185.42 86.36) (xy 185.42 81.28))
-    (stroke (width 0) (type default) (color 0 0 0 0))
-  )
-  (wire (pts (xy 156.21 78.74) (xy 142.24 78.74))
-    (stroke (width 0) (type default) (color 0 0 0 0))
-  )
   (wire (pts (xy 83.82 96.52) (xy 88.9 96.52))
     (stroke (width 0) (type default) (color 0 0 0 0))
@@
   )
   (wire (pts (xy 88.9 88.9) (xy 111.76 88.9))
-    (stroke (width 0) (type default) (color 0 0 0 0))
-  )
-  (wire (pts (xy 100.33 73.66) (xy 100.33 78.74))
     (stroke (width 0) (type default) (color 0 0 0 0))
   )
@@
     (effects (font (size 1.27 1.27)) (justify left))
   )
-  (hierarchical_label "Vcc" (shape input) (at 100.33 73.66 90)
+  (hierarchical_label "Vcc" (shape input) (at 100.33 63.5 90)
     (effects (font (size 1.27 1.27)) (justify left))
   )
@@
     (in_bom yes) (on_board yes)
     (property "Reference" "R203" (id 0) (at 104.14 76.2 90))
-    (property "Value" "47k" (id 1) (at 104.14 78.74 90))
+    (property "Value" "10k" (id 1) (at 104.14 78.74 90))
     (property "Footprint" "Resistor_SMD:R_0805_2012Metric_Pad1.20x1.40mm_HandSolder" (id 2) (at 104.14 80.518 90)
       (effects (font (size 1.27 1.27)) hide)
@@
     (in_bom yes) (on_board yes)
     (property "Reference" "R204" (id 0) (at 104.14 81.28 90))
-    (property "Value" "47k" (id 1) (at 104.14 83.82 90))
+    (property "Value" "10k" (id 1) (at 104.14 83.82 90))
     (property "Footprint" "Resistor_SMD:R_0805_2012Metric_Pad1.20x1.40mm_HandSolder" (id 2) (at 104.14 85.598 90)
       (effects (font (size 1.27 1.27)) hide)
@@
     (in_bom yes) (on_board yes)
     (property "Reference" "R205" (id 0) (at 153.67 74.93 90))
-    (property "Value" "47k" (id 1) (at 156.21 74.93 90))
+    (property "Value" "10k" (id 1) (at 156.21 74.93 90))
     (property "Footprint" "Resistor_SMD:R_0805_2012Metric_Pad1.20x1.40mm_HandSolder" (id 2) (at 157.988 74.93 90)
       (effects (font (size 1.27 1.27)) hide)
@@
     (in_bom yes) (on_board yes)
     (property "Reference" "R206" (id 0) (at 153.67 105.41 90))
-    (property "Value" "47k" (id 1) (at 156.21 105.41 90))
+    (property "Value" "10k" (id 1) (at 156.21 105.41 90))
     (property "Footprint" "Resistor_SMD:R_0805_2012Metric_Pad1.20x1.40mm_HandSolder" (id 2) (at 157.988 105.41 90)
       (effects (font (size 1.27 1.27)) hide)

Commit message: consolidating RST with EN and adding a capacitor for stability. fixes #1
Parts:
- removed R204: 10k, Resistor_SMD:R_0805_2012Metric_Pad1.20x1.40mm_HandSolder, symbol Device:R
- added C204: 100n, Capacitor_SMD:C_0805_2012Metric_Pad1.18x1.45mm_HandSolder, symbol Device:C
Connections:
- net _EN is gone; now on net _RST: U201.3 (EN)
- net Vcc: now also C204.2
- net _RST: now also C204.1
Other:
- moved on the sheet: R203
Changed lines of the file:
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@@
   (junction (at 156.21 101.6) (diameter 0) (color 0 0 0 0)
   )
+  (junction (at 107.95 64.77) (diameter 0) (color 0 0 0 0)
+  )
   (junction (at 156.21 78.74) (diameter 0) (color 0 0 0 0)
   )
@@
   (junction (at 83.82 88.9) (diameter 0) (color 0 0 0 0)
   )
-  (junction (at 100.33 78.74) (diameter 0) (color 0 0 0 0)
+  (junction (at 107.95 78.74) (diameter 0) (color 0 0 0 0)
+  )
+  (junction (at 107.95 72.39) (diameter 0) (color 0 0 0 0)
   )
   (junction (at 88.9 88.9) (diameter 0) (color 0 0 0 0)
@@
     (stroke (width 0) (type default) (color 0 0 0 0))
   )
+  (wire (pts (xy 107.95 72.39) (xy 107.95 78.74))
+    (stroke (width 0) (type default) (color 0 0 0 0))
+  )
+  (wire (pts (xy 107.95 72.39) (xy 115.57 72.39))
+    (stroke (width 0) (type default) (color 0 0 0 0))
+  )
   (wire (pts (xy 158.75 93.98) (xy 142.24 93.98))
     (stroke (width 0) (type default) (color 0 0 0 0))
@@
     (stroke (width 0) (type default) (color 0 0 0 0))
   )
-  (wire (pts (xy 107.95 83.82) (xy 111.76 83.82))
+  (wire (pts (xy 107.95 64.77) (xy 115.57 64.77))
     (stroke (width 0) (type default) (color 0 0 0 0))
   )
@@
     (stroke (width 0) (type default) (color 0 0 0 0))
   )
-  (wire (pts (xy 100.33 63.5) (xy 100.33 78.74))
+  (wire (pts (xy 107.95 62.23) (xy 107.95 64.77))
     (stroke (width 0) (type default) (color 0 0 0 0))
   )
@@
     (stroke (width 0) (type default) (color 0 0 0 0))
   )
+  (wire (pts (xy 111.76 83.82) (xy 107.95 83.82))
+    (stroke (width 0) (type default) (color 0 0 0 0))
+  )
   (wire (pts (xy 88.9 88.9) (xy 111.76 88.9))
     (stroke (width 0) (type default) (color 0 0 0 0))
   )
-  (wire (pts (xy 100.33 78.74) (xy 100.33 83.82))
-    (stroke (width 0) (type default) (color 0 0 0 0))
-  )
   (wire (pts (xy 130.81 66.04) (xy 140.97 66.04))
+    (stroke (width 0) (type default) (color 0 0 0 0))
+  )
+  (wire (pts (xy 107.95 83.82) (xy 107.95 78.74))
     (stroke (width 0) (type default) (color 0 0 0 0))
   )
@@
     (effects (font (size 0.5 0.5)) (justify left bottom))
   )
-  (label "_EN" (at 109.22 83.82 0)
-    (effects (font (size 0.5 0.5)) (justify left bottom))
-  )
   (label "_RX" (at 142.24 86.36 0)
     (effects (font (size 0.5 0.5)) (justify left bottom))
@@
     (effects (font (size 1.27 1.27)) (justify left))
   )
-  (hierarchical_label "Vcc" (shape input) (at 100.33 63.5 90)
+  (hierarchical_label "Vcc" (shape input) (at 107.95 62.23 90)
     (effects (font (size 1.27 1.27)) (justify left))
   )
@@
     (pin "2")
   )
-  (symbol (lib_id "Device:R") (at 104.14 78.74 90) (unit 1)
-    (in_bom yes) (on_board yes)
-    (property "Reference" "R203" (id 0) (at 104.14 76.2 90))
-    (property "Value" "10k" (id 1) (at 104.14 78.74 90))
-    (property "Footprint" "Resistor_SMD:R_0805_2012Metric_Pad1.20x1.40mm_HandSolder" (id 2) (at 104.14 80.518 90)
-      (effects (font (size 1.27 1.27)) hide)
-    )
-    (property "Datasheet" "~" (id 3) (at 104.14 78.74 0)
+  (symbol (lib_id "Device:C") (at 115.57 68.58 180) (unit 1)
+    (in_bom yes) (on_board yes)
+    (property "Reference" "C204" (id 0) (at 116.84 66.04 0)
+      (effects (font (size 1.27 1.27)) (justify right))
+    )
+    (property "Value" "100n" (id 1) (at 116.84 71.12 0)
+      (effects (font (size 1.27 1.27)) (justify right))
+    )
+    (property "Footprint" "Capacitor_SMD:C_0805_2012Metric_Pad1.18x1.45mm_HandSolder" (id 2) (at 114.6048 64.77 0)
+      (effects (font (size 1.27 1.27)) hide)
+    )
+    (property "Datasheet" "~" (id 3) (at 115.57 68.58 0)
+      (effects (font (size 1.27 1.27)) hide)
+    )
+    (pin "1")
+    (pin "2")
+  )
+  (symbol (lib_id "Device:R") (at 107.95 68.58 0) (unit 1)
+    (in_bom yes) (on_board yes)
+    (property "Reference" "R203" (id 0) (at 110.49 68.58 90))
+    (property "Value" "10k" (id 1) (at 107.95 68.58 90))
+    (property "Footprint" "Resistor_SMD:R_0805_2012Metric_Pad1.20x1.40mm_HandSolder" (id 2) (at 106.172 68.58 90)
+      (effects (font (size 1.27 1.27)) hide)
+    )
+    (property "Datasheet" "~" (id 3) (at 107.95 68.58 0)
       (effects (font (size 1.27 1.27)) hide)
     )
@@
       (effects (font (size 1.27 1.27)) hide)
     )
-    (pin "1")
-    (pin "2")
-  )
-  (symbol (lib_id "Device:R") (at 104.14 83.82 90) (unit 1)
-    (in_bom yes) (on_board yes)
-    (property "Reference" "R204" (id 0) (at 104.14 81.28 90))
-    (property "Value" "10k" (id 1) (at 104.14 83.82 90))
-    (property "Footprint" "Resistor_SMD:R_0805_2012Metric_Pad1.20x1.40mm_HandSolder" (id 2) (at 104.14 85.598 90)
-      (effects (font (size 1.27 1.27)) hide)
-    )
-    (property "Datasheet" "~" (id 3) (at 104.14 83.82 0)
-      (effects (font (size 1.27 1.27)) hide)
-    )
