File: project/_psu.kicad_sch (KiCad schematic)
At the start: 23 parts, among them Q301 AO3401A, Q302 AO3401A, SW301 SW_SPDT, SW302 btn, U301 BMS_USB_LiPo_Charger, U302 TPL5110

Commit message: various small improvements
Parts:
- SW301: footprint Button_Switch_SMD:SW_SPDT_PCM12 -> -local:SW_SPDT_PCM12; symbol Switch:SW_SPDT -> -modules:SW_SPDT
Connections:
- net GND: now also SW301.MP
- net Vusb renamed _vusb
Other:
- moved on the sheet: R304, R305

Commit message: fixing bom, datasheets and adding link to repo
Parts:
- BT301: LCSC Part Number (none) -> C2988620; MPN (none) -> BH-18650-B1BA002
- C303, C304: LCSC Part Number (none) -> C312983; MPN (none) -> GRM31CR61A107ME05L
- F301: value 1A -> PTC 1A; LCSC Part Number (none) -> C2830246; MPN (none) -> JK-nSMD100/16V
- Q301, Q302: LCSC Part Number (none) -> C347476; MPN (none) -> AO3401A
- SW301: LCSC Part Number (none) -> C431540; MPN (none) -> MSK12C02
- U302: LCSC Part Number (none) -> C125830; MPN (none) -> TPL5110
Changed lines of the file:
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@@
   (title_block
     (title "WiScale")
-    (date "2022-11-14")
+    (date "2022-11-24")
     (rev "1.0")
   )
@@
       (effects (font (size 1.27 1.27)) (justify left) hide)
     )
+    (property "LCSC Part Number" "C347476" (id 4) (at 226.06 90.17 0)
+      (effects (font (size 1.27 1.27)) hide)
+    )
+    (property "MPN" "AO3401A" (id 5) (at 226.06 90.17 0)
+      (effects (font (size 1.27 1.27)) hide)
+    )
     (pin "1")
     (pin "2")
@@
   (symbol (lib_id "power:GND") (at 182.88 114.3 0) (unit 1)
     (in_bom yes) (on_board yes)
-    (property "Reference" "#PWR?" (id 0) (at 182.88 120.65 0)
+    (property "Reference" "#PWR0102" (id 0) (at 182.88 120.65 0)
       (effects (font (size 1.27 1.27)) hide)
     )
@@
       (effects (font (size 1.27 1.27)) hide)
     )
-    (property "Datasheet" "~" (id 3) (at 170.18 91.44 0)
+    (property "Datasheet" "https://datasheet.lcsc.com/lcsc/1811061115_Murata-Electronics-GRM31CR61A107ME05L_C312983.pdf" (id 3) (at 170.18 91.44 0)
+      (effects (font (size 1.27 1.27)) hide)
+    )
+    (property "LCSC Part Number" "C312983" (id 4) (at 170.18 91.44 0)
+      (effects (font (size 1.27 1.27)) hide)
+    )
+    (property "MPN" "GRM31CR61A107ME05L" (id 5) (at 170.18 91.44 0)
       (effects (font (size 1.27 1.27)) hide)
     )
@@
       (effects (font (size 1.27 1.27)) (justify left) hide)
     )
+    (property "LCSC Part Number" "C347476" (id 4) (at 101.6 96.52 0)
+      (effects (font (size 1.27 1.27)) hide)
+    )
+    (property "MPN" "AO3401A" (id 5) (at 101.6 96.52 0)
+      (effects (font (size 1.27 1.27)) hide)
+    )
     (pin "1")
     (pin "2")
@@
     (in_bom yes) (on_board yes)
     (property "Reference" "F301" (id 0) (at 116.84 91.44 90))
-    (property "Value" "1A" (id 1) (at 119.38 96.52 90))
+    (property "Value" "PTC 1A" (id 1) (at 119.38 96.52 90))
     (property "Footprint" "Fuse:Fuse_1206_3216Metric_Pad1.42x1.75mm_HandSolder" (id 2) (at 123.19 92.71 0)
       (effects (font (size 1.27 1.27)) (justify left) hide)
     )
-    (property "Datasheet" "~" (id 3) (at 118.11 93.98 0)
+    (property "Datasheet" "https://datasheet.lcsc.com/lcsc/2105241640_Jinrui-Electronic-Materials-Co--JK-nSMD100-16V_C2830246.pdf" (id 3) (at 118.11 93.98 0)
+      (effects (font (size 1.27 1.27)) hide)
+    )
+    (property "LCSC Part Number" "C2830246" (id 4) (at 118.11 93.98 0)
+      (effects (font (size 1.27 1.27)) hide)
+    )
+    (property "MPN" "JK-nSMD100/16V" (id 5) (at 118.11 93.98 0)
       (effects (font (size 1.27 1.27)) hide)
     )
@@
     )
     (property "Datasheet" "http://www.ti.com/lit/ds/symlink/tpl5110.pdf" (id 3) (at 205.74 114.3 0)
+      (effects (font (size 1.27 1.27)) hide)
+    )
+    (property "LCSC Part Number" "C125830" (id 4) (at 210.82 104.14 0)
+      (effects (font (size 1.27 1.27)) hide)
+    )
+    (property "MPN" "TPL5110" (id 5) (at 210.82 104.14 0)
       (effects (font (size 1.27 1.27)) hide)
     )
@@
       (effects (font (size 1.27 1.27)) hide)
     )
-    (property "Datasheet" "~" (id 3) (at 180.34 109.22 0)
+    (property "Datasheet" "https://datasheet.lcsc.com/lcsc/1912111437_SHOU-HAN-MSK12C02_C431540.pdf" (id 3) (at 180.34 109.22 0)
+      (effects (font (size 1.27 1.27)) hide)
+    )
+    (property "LCSC Part Number" "C431540" (id 4) (at 180.34 109.22 0)
+      (effects (font (size 1.27 1.27)) hide)
+    )
+    (property "MPN" "MSK12C02" (id 5) (at 180.34 109.22 0)
       (effects (font (size 1.27 1.27)) hide)
     )
@@
       (effects (font (size 1.27 1.27)) hide)
     )
-    (property "Datasheet" "~" (id 3) (at 125.73 97.536 90)
+    (property "Datasheet" "https://datasheet.lcsc.com/lcsc/2204021730_MYOUNG-BH-18650-B1BA002_C2988620.pdf" (id 3) (at 125.73 97.536 90)
+      (effects (font (size 1.27 1.27)) hide)
+    )
+    (property "LCSC Part Number" "C2988620" (id 4) (at 125.73 99.06 0)
+      (effects (font (size 1.27 1.27)) hide)
+    )
+    (property "MPN" "BH-18650-B1BA002" (id 5) (at 125.73 99.06 0)
       (effects (font (size 1.27 1.27)) hide)
     )
@@
       (effects (font (size 1.27 1.27)) hide)
     )
-    (property "Datasheet" "~" (id 3) (at 177.8 91.44 0)
-      (effects (font (size 1.27 1.27)) hide)
-    )
+    (property "Datasheet" "https://datasheet.lcsc.com/lcsc/1811061115_Murata-Electronics-GRM31CR61A107ME05L_C312983.pdf" (id 3) (at 177.8 91.44 0)
+      (effects (font (size 1.27 1.27)) hide)
+    )
+    (property "LCSC Part Number" "C312983" (id 4) (at 177.8 91.44 0)
+      (effects (font (size 1.27 1.27)) hide)
+    )
+    (property "MPN" "GRM31CR61A107ME05L" (id 5) (at 177.8 91.44 0)
+      (effects (font (size 1.27 1.27)) hide)
+    )

Commit message: adding usb port with ldo and diode options
Parts:
- added C307, C308: 10u, Capacitor_SMD:C_0805_2012Metric_Pad1.18x1.45mm_HandSolder, symbol Device:C
- added D301, D302: 1N4148WL, Diode_SMD:D_SOD-123, symbol Diode:1N4148W
- added D303: GREEN, LED_SMD:LED_0805_2012Metric_Pad1.15x1.40mm_HandSolder, symbol Device:LED
- added J301: USB_POWER_IN, -local:USB_C_Receptacle_HRO_TYPE-C-31-M-12, symbol Connector:USB_C_Receptacle_USB2.0
- added R309, R310, R311: 4k7, Resistor_SMD:R_0805_2012Metric_Pad1.20x1.40mm_HandSolder, symbol Device:R
- added U303: AMS1117-3.3, Package_TO_SOT_SMD:SOT-223-3_TabPin2, symbol Regulator_Linear:AMS1117-3.3
Connections:
- net GND: now also C307.1, C308.1, D303.1 (K), J301.A1 (GND), J301.A12 (GND), J301.B1 (GND), J301.B12 (GND), J301.S1 (SHIELD), R309.1, R310.1, U303.1 (GND)
- net Vbat: now also C308.2, D302.1 (K), U303.2 (VO)
- net Vcc: now also R311.2
- new net: D301.1 (K), D302.2 (A)
- new net: D303.2 (A), R311.1
- new net _cc1: J301.A5 (CC1), R310.2
- new net _cc2: J301.B5 (CC2), R309.2
- new net _usb_vbus: C307.2, D301.2 (A), J301.A4 (VBUS), J301.A9 (VBUS), J301.B4 (VBUS), J301.B9 (VBUS), U303.3 (VI)
- no-connect marks 0 -> 6

Commit message: fixing charging detection divider, fixes #2
Connections:
- net Charging: now also R301.1, R302.2; no longer R301.2
- net _vusb: now also R301.2; no longer R301.1, R302.2
Other:
- moved on the sheet: BT301, BT302, C301, C302, C303, C304, C305, C306, C307, C308, D301, D302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

Commit message: connected LDO USB power with charger USB power, fixes #3
Connections:
- net _vusb is gone; now on net Vusb: R301.2, U301.i1 (IN+)
- net _usb_vbus renamed Vusb
Changed lines of the file:
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@@
   (junction (at 127 67.31) (diameter 0) (color 0 0 0 0)
   )
-  (junction (at 93.98 100.33) (diameter 0) (color 0 0 0 0)
-  )
   (junction (at 109.22 59.69) (diameter 0) (color 0 0 0 0)
   )
@@
   (junction (at 195.58 53.34) (diameter 0) (color 0 0 0 0)
   )
-  (junction (at 49.53 59.69) (diameter 0) (color 0 0 0 0)
-  )
   (junction (at 232.41 53.34) (diameter 0) (color 0 0 0 0)
   )
   (junction (at 113.03 107.95) (diameter 0) (color 0 0 0 0)
+  )
+  (junction (at 53.34 59.69) (diameter 0) (color 0 0 0 0)
+  )
+  (junction (at 83.82 100.33) (diameter 0) (color 0 0 0 0)
   )
   (no_connect (at 83.82 130.81))
@@
     (stroke (width 0) (type default) (color 0 0 0 0))
   )
+  (wire (pts (xy 83.82 90.17) (xy 83.82 100.33))
+    (stroke (width 0) (type default) (color 0 0 0 0))
+  )
   (wire (pts (xy 113.03 107.95) (xy 127 107.95))
     (stroke (width 0) (type default) (color 0 0 0 0))
@@
     (stroke (width 0) (type default) (color 0 0 0 0))
   )
-  (wire (pts (xy 88.9 100.33) (xy 93.98 100.33))
-    (stroke (width 0) (type default) (color 0 0 0 0))
-  )
   (wire (pts (xy 231.14 44.45) (xy 232.41 44.45))
     (stroke (width 0) (type default) (color 0 0 0 0))
   )
-  (wire (pts (xy 49.53 59.69) (xy 55.88 59.69))
+  (wire (pts (xy 46.99 59.69) (xy 53.34 59.69))
     (stroke (width 0) (type default) (color 0 0 0 0))
   )
@@
     (stroke (width 0) (type default) (color 0 0 0 0))
   )
-  (wire (pts (xy 93.98 100.33) (xy 99.06 100.33))
+  (wire (pts (xy 88.9 100.33) (xy 99.06 100.33))
     (stroke (width 0) (type default) (color 0 0 0 0))
   )
@@
     (stroke (width 0) (type default) (color 0 0 0 0))
   )
+  (wire (pts (xy 53.34 59.69) (xy 55.88 59.69))
+    (stroke (width 0) (type default) (color 0 0 0 0))
+  )
   (wire (pts (xy 123.19 59.69) (xy 127 59.69))
     (stroke (width 0) (type default) (color 0 0 0 0))
@@
     (stroke (width 0) (type default) (color 0 0 0 0))
   )
+  (wire (pts (xy 53.34 50.8) (xy 53.34 59.69))
+    (stroke (width 0) (type default) (color 0 0 0 0))
+  )
   (wire (pts (xy 109.22 59.69) (xy 107.95 59.69))
     (stroke (width 0) (type default) (color 0 0 0 0))
@@
   )
   (wire (pts (xy 88.9 86.36) (xy 88.9 100.33))
-    (stroke (width 0) (type default) (color 0 0 0 0))
-  )
-  (wire (pts (xy 46.99 59.69) (xy 49.53 59.69))
     (stroke (width 0) (type default) (color 0 0 0 0))
   )
@@
     (effects (font (size 0.5 0.5)) (justify left bottom))
   )
-  (label "_usb_vbus" (at 83.82 100.33 0)
-    (effects (font (size 0.5 0.5)) (justify left bottom))
-  )
   (label "_delay" (at 195.58 72.39 0)
     (effects (font (size 0.5 0.5)) (justify left bottom))
@@
   (label "_drv_gate" (at 227.33 69.85 0)
     (effects (font (size 0.5 0.5)) (justify left bottom))
-  )
-  (label "_vusb" (at 55.88 59.69 180)
-    (effects (font (size 1.27 1.27)) (justify right bottom))
   )
   (label "_cc1" (at 83.8807 105.41 0)
@@
     (pin "2")
   )
+  (symbol (lib_id "-pwr:Vusb") (at 166.37 182.88 0) (unit 1)
+    (in_bom yes) (on_board yes) (fields_autoplaced)
+    (property "Reference" "#PWR0105" (id 0) (at 166.37 186.69 0)
+      (effects (font (size 1.27 1.27)) hide)
+    )
+    (property "Value" "Vusb" (id 1) (at 166.37 177.8 0))
+    (property "Footprint" "" (id 2) (at 166.37 182.88 0)
+      (effects (font (size 1.27 1.27)) hide)
+    )
+    (property "Datasheet" "" (id 3) (at 166.37 182.88 0)
+      (effects (font (size 1.27 1.27)) hide)
+    )
+    (pin "1")
+  )
   (symbol (lib_id "Transistor_FET:AO3401A") (at 102.87 62.23 270) (mirror x) (unit 1)
     (in_bom yes) (on_board yes)
@@
     (pin "1")
   )
+  (symbol (lib_id "-pwr:Vusb") (at 83.82 90.17 0) (unit 1)
+    (in_bom yes) (on_board yes)
+    (property "Reference" "#PWR0103" (id 0) (at 83.82 93.98 0)
+      (effects (font (size 1.27 1.27)) hide)
+    )
+    (property "Value" "Vusb" (id 1) (at 83.82 86.36 0))
+    (property "Footprint" "" (id 2) (at 83.82 90.17 0)
+      (effects (font (size 1.27 1.27)) hide)
+    )
+    (property "Datasheet" "" (id 3) (at 83.82 90.17 0)
+      (effects (font (size 1.27 1.27)) hide)
+    )
+    (pin "1")
+  )
   (symbol (lib_id "Device:R") (at 227.33 44.45 90) (unit 1)
     (in_bom yes) (on_board yes)
@@
     (pin "1")
     (pin "2")
-  )
-  (symbol (lib_id "power:PWR_FLAG") (at 93.98 100.33 0) (unit 1)
-    (in_bom yes) (on_board yes)
-    (property "Reference" "#FLG0103" (id 0) (at 93.98 98.425 0)
-      (effects (font (size 1.27 1.27)) hide)
-    )
-    (property "Value" "PWR_FLAG" (id 1) (at 90.17 96.52 0)
-      (effects (font (size 1.27 1.27)) (justify left))
-    )
-    (property "Footprint" "" (id 2) (at 93.98 100.33 0)
-      (effects (font (size 1.27 1.27)) hide)
-    )
-    (property "Datasheet" "~" (id 3) (at 93.98 100.33 0)
-      (effects (font (size 1.27 1.27)) hide)
-    )
-    (pin "1")
   )
   (symbol (lib_id "Timer:TPL5110") (at 212.09 69.85 0) (unit 1)
@@
     (pin "1")
   )
+  (symbol (lib_id "-pwr:Vusb") (at 53.34 50.8 0) (unit 1)
+    (in_bom yes) (on_board yes)
+    (property "Reference" "#PWR0104" (id 0) (at 53.34 54.61 0)
+      (effects (font (size 1.27 1.27)) hide)
+    )
+    (property "Value" "Vusb" (id 1) (at 53.34 46.99 0))
+    (property "Footprint" "" (id 2) (at 53.34 50.8 0)
+      (effects (font (size 1.27 1.27)) hide)
+    )
+    (property "Datasheet" "" (id 3) (at 53.34 50.8 0)
+      (effects (font (size 1.27 1.27)) hide)
+    )
+    (pin "1")
+  )
   (symbol (lib_id "Device:R") (at 88.9 115.57 180) (unit 1)
     (in_bom yes) (on_board yes)
@@
     (pin "2")
   )
-  (symbol (lib_id "power:PWR_FLAG") (at 49.53 59.69 0) (unit 1)
-    (in_bom yes) (on_board yes)
-    (property "Reference" "#FLG0102" (id 0) (at 49.53 57.785 0)
-      (effects (font (size 1.27 1.27)) hide)
-    )
-    (property "Value" "PWR_FLAG" (id 1) (at 46.99 55.88 0)
+  (symbol (lib_id "power:PWR_FLAG") (at 166.37 182.88 180) (unit 1)
+    (in_bom yes) (on_board yes)
+    (property "Reference" "#FLG0102" (id 0) (at 166.37 184.785 0)
+      (effects (font (size 1.27 1.27)) hide)
+    )
+    (property "Value" "PWR_FLAG" (id 1) (at 168.91 186.69 0)
       (effects (font (size 1.27 1.27)) (justify left))
     )
-    (property "Footprint" "" (id 2) (at 49.53 59.69 0)
-      (effects (font (size 1.27 1.27)) hide)
-    )
-    (property "Datasheet" "~" (id 3) (at 49.53 59.69 0)
-      (effects (font (size 1.27 1.27)) hide)
-    )
+    (property "Footprint" "" (id 2) (at 166.37 182.88 0)
+      (effects (font (size 1.27 1.27)) hide)
+    )
+    (property "Datasheet" "~" (id 3) (at 166.37 182.88 0)
+      (effects (font (size 1.27 1.27)) hide)
+    )
