File: project/_temp.kicad_sch (KiCad schematic)
At the start: 4 parts, among them J801 DS18B20, U801 DS18B20Z, U802 DS18B20

Commit message: fixing bom, datasheets and adding link to repo
Other:
- title: (none) -> WiScale
Changed lines of the file:
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@@
 (kicad_sch (version 20211123) (generator eeschema)
   (paper "A4")
+  (title_block
+    (title "WiScale")
+    (date "2022-11-24")
+    (rev "1.0")
+  )
   (wire (pts (xy 142.24 109.22) (xy 139.7 109.22))
     (stroke (width 0) (type default) (color 0 0 0 0))
